File: Mosaic System templates V1.00 12-2022/MM 50x50/MM 50x50 template.kicad_pcb (KiCad board)
At the start: 2 copper layers, 50 x 50 mm, 3 parts

Commit message: V1
Parts:
- moved REF3 35.0 mm to (150.0, 100.0)
Changed lines of the file:
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@@
       (layer "F.SilkS" (type "Top Silk Screen") (color "White"))
       (layer "F.Paste" (type "Top Solder Paste"))
-      (layer "F.Mask" (type "Top Solder Mask") (color "Black") (thickness 0.01))
+      (layer "F.Mask" (type "Top Solder Mask") (color "#000000FF") (thickness 0.01))
       (layer "F.Cu" (type "copper") (thickness 0.035))
       (layer "dielectric 1" (type "core") (thickness 1.51) (material "FR4") (epsilon_r 4.5) (loss_tangent 0.02))
       (layer "B.Cu" (type "copper") (thickness 0.035))
-      (layer "B.Mask" (type "Bottom Solder Mask") (color "Black") (thickness 0.01))
+      (layer "B.Mask" (type "Bottom Solder Mask") (color "#000000FF") (thickness 0.01))
       (layer "B.Paste" (type "Bottom Solder Paste"))
       (layer "B.SilkS" (type "Bottom Silk Screen") (color "White"))
@@
   )
   (footprint "0-MM:MM_LOGO" (layer "F.Cu")
-    (at 150 135)
+    (at 150 100)
     (property "Sheetfile" "")
     (property "Sheetname" "")
